Commit message: Update meshes for tiago dual arm

File: tiago_dual_description/urdf/torso/torso_dual.urdf.xacro (robot description, xacro)
@@ -27,5 +27,5 @@
       <origin rpy="0 0 0" xyz="0 0 0" />
       <geometry>
-        <mesh filename="package://tiago_description/meshes/torso/torso_fix.stl" scale="1 1 1"/>
+        <mesh filename="package://tiago_dual_description/meshes/torso/torso_fix.stl" scale="1 1 1"/>
       </geometry>
       <material name="LightGrey"/>
@@ -95,5 +95,5 @@
       <origin rpy="0 0 0" xyz="0 0 0" />
        <geometry>
-        <mesh filename="package://tiago_description/meshes/torso/torso_lift_with_arm.stl" scale="1 1 1"/>
+        <mesh filename="package://tiago_dual_description/meshes/torso/torso_lift_dual_arm.stl" scale="1 1 1"/>
       </geometry>
       <material name="White"/>
@@ -106,6 +106,15 @@
       <material name="LightGrey"/>
     </collision>
+    <!-- left shoulder collision-->
     <collision>
-      <origin rpy="0 0 0" xyz="0 0 0" />
+      <origin rpy="0 0 0" xyz="-0.131 0.17 -0.02556" />
+       <geometry>
+        <mesh filename="package://tiago_description/meshes/torso/torso_lift_collision_shoulder.dae" scale="1 1 1"/>
+      </geometry>
+      <material name="LightGrey"/>
+    </collision>
+    <!-- right shoulder collision-->
+    <collision>
+      <origin rpy="0 0 0" xyz="-0.131 -0.19 -0.02556" />
        <geometry>
         <mesh filename="package://tiago_description/meshes/torso/torso_lift_collision_shoulder.dae" scale="1 1 1"/>

Commit message: Fix collision boxes for the torso

File: tiago_dual_description/urdf/torso/torso_dual.urdf.xacro (robot description, xacro)
@@ -34,5 +34,5 @@
       <origin rpy="0 0 0" xyz="0.085 0.0 0.02" />
       <geometry>
-        <box size="0.4 0.25 0.04"/>
+        <box size="0.4 0.265 0.057"/>
       </geometry>
     </collision>
@@ -40,5 +40,5 @@
       <origin rpy="0 0 0" xyz="0 0 0.05" />
       <geometry>
-        <box size="0.25 0.25 0.1"/>
+        <box size="0.25 0.265 0.052"/>
       </geometry>
     </collision>
@@ -69,5 +69,5 @@
       <origin rpy="0 0 0" xyz="0 0 0.275" />
       <geometry>
-        <box size="0.23 0.23 0.55"/>
+        <box size="0.232 0.26 0.45"/>
       </geometry>
       <material name="DarkGrey"/>

Commit message: Added if condition in torso xacro

File: tiago_dual_description/urdf/torso/torso_dual.urdf.xacro (robot description, xacro)
@@ -148,4 +148,12 @@
     </xacro:unless>
   </link>
+  <xacro:if value="$(arg fixed_torso)">
+  <joint name="${name}_lift_joint" type="fixed">
+    <origin rpy="0.0 0.0 0.0" xyz="0.0 0.0 0.597" />
+    <parent link="${name}_fixed_link" />
+    <child link="${name}_lift_link" />
+  </joint>
+</xacro:if>
+<xacro:unless value="$(arg fixed_torso)">
   <joint name="${name}_lift_joint" type="prismatic">
     <origin rpy="0.0 0.0 0.0" xyz="0.0 0.0 0.597" />
@@ -157,9 +165,10 @@
     <dynamics damping="1000" />
     <safety_controller k_position="20"
-                         k_velocity="20"
-                         soft_lower_limit="0.0"
-                         soft_upper_limit="0.35" />
+      k_velocity="20"
+      soft_lower_limit="0.0"
+      soft_upper_limit="0.35" />
   </joint>
-  <xacro:torso_simple_transmission name="torso_lift" reduction="1.0"/>
+  <xacro:torso_simple_transmission name="torso_lift" reduction="1.0" />
+</xacro:unless>
  </xacro:macro>
 </robot>

Commit message: Manual formating

File: tiago_dual_description/urdf/torso/torso_dual.urdf.xacro (robot description, xacro)
@@ -149,26 +149,26 @@
   </link>
   <xacro:if value="$(arg fixed_torso)">
-  <joint name="${name}_lift_joint" type="fixed">
-    <origin rpy="0.0 0.0 0.0" xyz="0.0 0.0 0.597" />
-    <parent link="${name}_fixed_link" />
-    <child link="${name}_lift_link" />
-  </joint>
-</xacro:if>
-<xacro:unless value="$(arg fixed_torso)">
-  <joint name="${name}_lift_joint" type="prismatic">
-    <origin rpy="0.0 0.0 0.0" xyz="0.0 0.0 0.597" />
-    <parent link="${name}_fixed_link" />
-    <child link="${name}_lift_link" />
-    <axis xyz="0 0 1" />
-    <limit effort="2000" lower="0" upper="0.35" velocity="${torso_max_vel}" />
-    <calibration rising="0.0" />
-    <dynamics damping="1000" />
-    <safety_controller k_position="20"
-      k_velocity="20"
-      soft_lower_limit="0.0"
-      soft_upper_limit="0.35" />
-  </joint>
-  <xacro:torso_simple_transmission name="torso_lift" reduction="1.0" />
-</xacro:unless>
+    <joint name="${name}_lift_joint" type="fixed">
+      <origin rpy="0.0 0.0 0.0" xyz="0.0 0.0 0.597" />
+      <parent link="${name}_fixed_link" />
+      <child link="${name}_lift_link" />
+    </joint>
+  </xacro:if>
+  <xacro:unless value="$(arg fixed_torso)">
+    <joint name="${name}_lift_joint" type="prismatic">
+      <origin rpy="0.0 0.0 0.0" xyz="0.0 0.0 0.597" />
+      <parent link="${name}_fixed_link" />
+      <child link="${name}_lift_link" />
+      <axis xyz="0 0 1" />
+      <limit effort="2000" lower="0" upper="0.35" velocity="${torso_max_vel}" />
+      <calibration rising="0.0" />
+      <dynamics damping="1000" />
+      <safety_controller k_position="20"
+        k_velocity="20"
+        soft_lower_limit="0.0"
+        soft_upper_limit="0.35" />
+    </joint>
+    <xacro:torso_simple_transmission name="torso_lift" reduction="1.0" />
+  </xacro:unless>
  </xacro:macro>
 </robot>

Commit message: updated the torso to be at half it's range when fixed

File: tiago_dual_description/urdf/torso/torso_dual.urdf.xacro (robot description, xacro)
@@ -150,5 +150,6 @@
   <xacro:if value="$(arg fixed_torso)">
     <joint name="${name}_lift_joint" type="fixed">
-      <origin rpy="0.0 0.0 0.0" xyz="0.0 0.0 0.597" />
+      <!-- Torso fixed height is set to half it's range -->
+      <origin rpy="0.0 0.0 0.0" xyz="0.0 0.0 0.772" />
       <parent link="${name}_fixed_link" />
       <child link="${name}_lift_link" />

Commit message: Update launch files, show.launch working

File: tiago_dual_description/urdf/torso/torso_dual.urdf.xacro (robot description, xacro)
@@ -28,5 +28,5 @@
                izz="0.07699800000"/>
     </inertial>
-    <!-- <visual>
+    <visual>
       <origin rpy="0 0 0" xyz="0 0 0" />
       <geometry>
@@ -46,5 +46,5 @@
         <box size="0.25 0.265 0.052"/>
       </geometry>
-    </collision> -->
+    </collision>
   </link>
   <joint name="${name}_fixed_joint" type="fixed">
@@ -96,5 +96,5 @@
     </inertial>
     <!-- Lifting body -->
-    <!-- <xacro:if value="${has_screen}">
+    <xacro:if value="${has_screen}">
       <visual>
         <origin rpy="0 0 0" xyz="0 0 0" />
@@ -111,7 +111,7 @@
         <material name="LightGrey"/>
       </collision>
-    </xacro:if> -->
-    <!-- <xacro:unless value="${has_screen}"> -->
-    <!-- <visual>
+    </xacro:if>
+    <xacro:unless value="${has_screen}">
+    <visual>
       <origin rpy="0 0 0" xyz="0 0 0" />
         <geometry>
@@ -119,6 +119,6 @@
       </geometry>
       <material name="White"/>
-    </visual> -->
-    <!-- <collision>
+    </visual>
+    <collision>
       <origin rpy="0 0 0" xyz="0 0 0" />
         <geometry>
@@ -126,7 +126,7 @@
       </geometry>
       <material name="LightGrey"/>
-    </collision> -->
+    </collision>
       <!-- left shoulder collision-->
-      <!-- <collision>
+      <collision>
         <origin rpy="0 0 0" xyz="-0.131 0.17 -0.02556" />
          <geometry>
@@ -134,7 +134,7 @@
         </geometry>
         <material name="LightGrey"/>
-      </collision> -->
+      </collision>
       <!-- right shoulder collision-->
-      <!-- <collision>
+      <collision>
         <origin rpy="0 0 0" xyz="-0.131 -0.19 -0.02556" />
          <geometry>
@@ -149,6 +149,6 @@
         </geometry>
         <material name="LightGrey"/>
-      </collision> -->
-    <!-- </xacro:unless> -->
+      </collision>
+    </xacro:unless>
   </link>
     <joint name="${name}_lift_joint" type="prismatic">

Commit message: Update tiago_dual_description/urdf/torso/torso_dual.urdf.xacro

File: tiago_dual_description/urdf/torso/torso_dual.urdf.xacro (robot description, xacro)
@@ -31,7 +31,7 @@
     </visual>
     <collision>
-      <origin rpy="0 0 0" xyz="0.085 0.0 0.02" />
+      <origin rpy="0 0 0" xyz="0.105 0.0 0.04" />
       <geometry>
-        <box size="0.4 0.265 0.057"/>
+        <box size="0.4 0.3 0.1"/>
       </geometry>
     </collision>

Commit message: Slightly decrease size of updated collision link

File: tiago_dual_description/urdf/torso/torso_dual.urdf.xacro (robot description, xacro)
@@ -31,7 +31,7 @@
     </visual>
     <collision>
-      <origin rpy="0 0 0" xyz="0.105 0.0 0.04" />
+      <origin rpy="0 0 0" xyz="0.09 0.0 0.02" />
       <geometry>
-        <box size="0.4 0.3 0.1"/>
+        <box size="0.4 0.28 0.075"/>
       </geometry>
     </collision>
