Commit message: Add torso for 2 arms

File: tiago_dual_description/robots/tiago_dual.urdf.xacro (robot description, xacro)
@@ -57,5 +57,5 @@
   <xacro:include filename="$(find pmb2_description)/urdf/base/base_sensors.urdf.xacro" />
   <!-- Torso -->
-  <xacro:include filename="$(find tiago_description)/urdf/torso/torso.urdf.xacro" />
+  <xacro:include filename="$(find tiago_dual_description)/urdf/torso/torso_dual.urdf.xacro" />
   <!-- Arm -->
   <xacro:include filename="$(find tiago_description)/urdf/arm/arm.urdf.xacro" />
@@ -75,11 +75,7 @@
   <xacro:head name="head" parent="torso_lift_link" camera_model="$(arg camera_model)"/>
   <!-- Left -->
-  <joint name="torso_left_lift_joint" type="fixed">
-    <origin xyz="0 0.5 0" rpy="0 0 0"/>
-    <parent link="torso_lift_link" />
-    <child link="torso_left_lift_link"/>
-  </joint>
-  <link name="torso_left_lift_link"/>
-  <xacro:tiago_arm name="arm_left" parent="torso_left_lift_link" wrist_6_range="${wrist_left_6_range}"/>
+  <xacro:tiago_arm name="arm_left" parent="torso_lift_link" wrist_6_range="${wrist_left_6_range}">
+    <origin xyz="0.02556 0.2565 -0.171" rpy="0 0 ${0 * deg_to_rad}"/>
+  </xacro:tiago_arm>
   <xacro:if value="${has_ft_sensor_left}">
       <xacro:ft_sensor name="wrist_left" parent="arm_left_tool_link" />
@@ -87,11 +83,7 @@
   <xacro:tiago_end_effector name="${end_effector_left_name}" parent="${end_effector_left_link}" type="${end_effector_left}" reflect="-1"/>
   <!-- Right -->
-  <joint name="torso_left_right_joint" type="fixed">
-    <origin xyz="0 -0.5 0" rpy="0 0 0"/>
-    <parent link="torso_lift_link" />
-    <child link="torso_right_lift_link"/>
-  </joint>
-  <link name="torso_right_lift_link"/>
-  <xacro:tiago_arm name="arm_right" parent="torso_right_lift_link" wrist_6_range="${wrist_right_6_range}"/>
+  <xacro:tiago_arm name="arm_right" parent="torso_lift_link" wrist_6_range="${wrist_right_6_range}">
+    <origin xyz="0.02556 -0.2565 -0.171" rpy="0 0 ${180 * deg_to_rad}"/>
+  </xacro:tiago_arm>
   <xacro:if value="${has_ft_sensor_right}">
       <xacro:ft_sensor name="wrist_right" parent="arm_right_tool_link" />

Commit message: Fix xacro warnings

File: tiago_dual_description/robots/tiago_dual.urdf.xacro (robot description, xacro)
@@ -43,14 +43,14 @@
     <xacro:wrong_camera_model/>
   </xacro:if>
-   <property name="has_schunk_ft"           value="${ft_sensor == 'schunk-ft'}"/>
-   <property name="has_ft_sensor_left"      value="${ft_sensor_left == 'schunk-ft'}"/> <!-- This should be OR'ed with other FT sensors-->
-   <property name="has_ft_sensor_right"     value="${ft_sensor_right == 'schunk-ft'}"/> <!-- This should be OR'ed with other FT sensors-->
-   <property name="end_effector_left_link"       value="${'wrist_left_ft_tg ool_link' if has_ft_sensor_left else 'arm_left_tool_link'}"/>
-   <property name="end_effector_left_name"       value="${'hand_left' if end_effector_left == 'pal-hey5' else 'gripper_left'}"/>
-   <property name="end_effector_right_link"       value="${'wrist_right_ft_tool_link' if has_ft_sensor_right else 'arm_right_tool_link'}"/>
-   <property name="end_effector_right_name"       value="${'hand_right' if end_effector_right == 'pal-hey5' else 'gripper_right'}"/>
-   <property name="wrist_left_6_range"      value="${ 81 if has_ft_sensor_left else 90 }"/>
-   <property name="wrist_right_6_range"     value="${ 81 if has_ft_sensor_right else 90 }"/>
-   <property name="head_link_name"          value="head_2_link"/>
+   <xacro:property name="has_schunk_ft"           value="${ft_sensor == 'schunk-ft'}"/>
+   <xacro:property name="has_ft_sensor_left"      value="${ft_sensor_left == 'schunk-ft'}"/> <!-- This should be OR'ed with other FT sensors-->
+   <xacro:property name="has_ft_sensor_right"     value="${ft_sensor_right == 'schunk-ft'}"/> <!-- This should be OR'ed with other FT sensors-->
+   <xacro:property name="end_effector_left_link"       value="${'wrist_left_ft_tg ool_link' if has_ft_sensor_left else 'arm_left_tool_link'}"/>
+   <xacro:property name="end_effector_left_name"       value="${'hand_left' if end_effector_left == 'pal-hey5' else 'gripper_left'}"/>
+   <xacro:property name="end_effector_right_link"       value="${'wrist_right_ft_tool_link' if has_ft_sensor_right else 'arm_right_tool_link'}"/>
+   <xacro:property name="end_effector_right_name"       value="${'hand_right' if end_effector_right == 'pal-hey5' else 'gripper_right'}"/>
+   <xacro:property name="wrist_left_6_range"      value="${ 81 if has_ft_sensor_left else 90 }"/>
+   <xacro:property name="wrist_right_6_range"     value="${ 81 if has_ft_sensor_right else 90 }"/>
+   <xacro:property name="head_link_name"          value="head_2_link"/>
   <!-- The following included files set up definitions of parts of the robot body -->
   <!-- Base -->

Commit message: Continue creation of tiago_dual_robot

File: tiago_dual_description/robots/tiago_dual.urdf.xacro (robot description, xacro)
@@ -46,5 +46,5 @@
    <xacro:property name="has_ft_sensor_left"      value="${ft_sensor_left == 'schunk-ft'}"/> <!-- This should be OR'ed with other FT sensors-->
    <xacro:property name="has_ft_sensor_right"     value="${ft_sensor_right == 'schunk-ft'}"/> <!-- This should be OR'ed with other FT sensors-->
-   <xacro:property name="end_effector_left_link"       value="${'wrist_left_ft_tg ool_link' if has_ft_sensor_left else 'arm_left_tool_link'}"/>
+   <xacro:property name="end_effector_left_link"       value="${'wrist_left_ft_tool_link' if has_ft_sensor_left else 'arm_left_tool_link'}"/>
    <xacro:property name="end_effector_left_name"       value="${'hand_left' if end_effector_left == 'pal-hey5' else 'gripper_left'}"/>
    <xacro:property name="end_effector_right_link"       value="${'wrist_right_ft_tool_link' if has_ft_sensor_right else 'arm_right_tool_link'}"/>

Commit message: Finish dual arm urdf

File: tiago_dual_description/robots/tiago_dual.urdf.xacro (robot description, xacro)
@@ -75,6 +75,6 @@
   <xacro:head name="head" parent="torso_lift_link" camera_model="$(arg camera_model)"/>
   <!-- Left -->
-  <xacro:tiago_arm name="arm_left" parent="torso_lift_link" wrist_6_range="${wrist_left_6_range}">
-    <origin xyz="0.02556 0.2565 -0.171" rpy="0 0 ${0 * deg_to_rad}"/>
+  <xacro:tiago_arm name="arm_left" parent="torso_lift_link" wrist_6_range="${wrist_left_6_range}" reflect="-1">
+    <origin xyz="0.02556 0.2565 -0.171" rpy="${180 * deg_to_rad} 0 ${180 * deg_to_rad}"/>
   </xacro:tiago_arm>
   <xacro:if value="${has_ft_sensor_left}">
@@ -83,5 +83,5 @@
   <xacro:tiago_end_effector name="${end_effector_left_name}" parent="${end_effector_left_link}" type="${end_effector_left}" reflect="-1"/>
   <!-- Right -->
-  <xacro:tiago_arm name="arm_right" parent="torso_lift_link" wrist_6_range="${wrist_right_6_range}">
+  <xacro:tiago_arm name="arm_right" parent="torso_lift_link" wrist_6_range="${wrist_right_6_range}" reflect="1">
     <origin xyz="0.02556 -0.2565 -0.171" rpy="0 0 ${180 * deg_to_rad}"/>
   </xacro:tiago_arm>

Commit message: New torso inertia and fixed arm_1 "Y"

File: tiago_dual_description/robots/tiago_dual.urdf.xacro (robot description, xacro)
@@ -72,9 +72,9 @@
   <!-- Now we can start using the macros included above to define the actual robot -->
   <xacro:base_sensors name="base" laser_model="$(arg laser_model)" sonars="true" microphone="true"/>
-  <xacro:tiago_torso name="torso" parent="base_link"/>
+  <xacro:tiago_dual_torso name="torso" parent="base_link"/>
   <xacro:head name="head" parent="torso_lift_link" camera_model="$(arg camera_model)"/>
   <!-- Left -->
   <xacro:tiago_arm name="arm_left" parent="torso_lift_link" wrist_6_range="${wrist_left_6_range}" reflect="-1">
-    <origin xyz="0.02556 0.2565 -0.171" rpy="${180 * deg_to_rad} 0 ${180 * deg_to_rad}"/>
+    <origin xyz="0.02556 0.19 -0.171" rpy="${180 * deg_to_rad} 0 ${180 * deg_to_rad}"/>
   </xacro:tiago_arm>
   <xacro:if value="${has_ft_sensor_left}">
@@ -84,5 +84,5 @@
   <!-- Right -->
   <xacro:tiago_arm name="arm_right" parent="torso_lift_link" wrist_6_range="${wrist_right_6_range}" reflect="1">
-    <origin xyz="0.02556 -0.2565 -0.171" rpy="0 0 ${180 * deg_to_rad}"/>
+    <origin xyz="0.02556 -0.19 -0.171" rpy="0 0 ${180 * deg_to_rad}"/>
   </xacro:tiago_arm>
   <xacro:if value="${has_ft_sensor_right}">

File: tiago_dual_description/urdf/torso/torso_dual.urdf.xacro (robot description, xacro)
@@ -14,5 +14,5 @@
   <xacro:property name="torso_max_vel"  value="0.07" />
   <xacro:property name="torso_eps"      value="0.02" />
-  <xacro:macro name="tiago_torso" params="name parent">
+  <xacro:macro name="tiago_dual_torso" params="name parent">
   <!-- Bottom fixed part of column -->
   <link name="${name}_fixed_link">
@@ -86,8 +86,8 @@
     <inertial>
       <origin xyz="0.04361 -0.00116 -0.17334" rpy="0.00000 0.00000 0.00000"/>
-      <mass value="8.166474"/>
-      <inertia ixx="0.271900" ixy="-0.001130" ixz="-0.009651"
-               iyy="0.188381" iyz="0.009095"
-               izz="0.135893"/>
+      <mass value="9.594213"/>
+      <inertia ixx="0.326395" ixy="-0.000844" ixz="-0.018905"
+               iyy="0.235332" iyz="0.009042"
+               izz="0.176168"/>
     </inertial>
     <!-- Lifting body -->

Commit message: Update description to match hardware changes

File: tiago_dual_description/robots/tiago_dual.urdf.xacro (robot description, xacro)
@@ -75,6 +75,6 @@
   <xacro:head name="head" parent="torso_lift_link" camera_model="$(arg camera_model)"/>
   <!-- Left -->
-  <xacro:tiago_arm name="arm_left" parent="torso_lift_link" wrist_6_range="${wrist_left_6_range}" reflect="-1">
-    <origin xyz="0.02556 0.19 -0.171" rpy="${180 * deg_to_rad} 0 ${180 * deg_to_rad}"/>
+  <xacro:tiago_arm name="arm_left" parent="torso_lift_link" wrist_6_range="${wrist_left_6_range}" reflect="-1" tiago_dual="1">
+    <origin xyz="0.02556 0.19 -0.171" rpy="${180 * deg_to_rad} 0 ${90 * deg_to_rad}"/>
   </xacro:tiago_arm>
   <xacro:if value="${has_ft_sensor_left}">
@@ -83,6 +83,6 @@
   <xacro:tiago_end_effector name="${end_effector_left_name}" parent="${end_effector_left_link}" type="${end_effector_left}" reflect="-1"/>
   <!-- Right -->
-  <xacro:tiago_arm name="arm_right" parent="torso_lift_link" wrist_6_range="${wrist_right_6_range}" reflect="1">
-    <origin xyz="0.02556 -0.19 -0.171" rpy="0 0 ${180 * deg_to_rad}"/>
+  <xacro:tiago_arm name="arm_right" parent="torso_lift_link" wrist_6_range="${wrist_right_6_range}" reflect="1" tiago_dual="1">
+    <origin xyz="0.02556 -0.19 -0.171" rpy="0 0 ${-90 * deg_to_rad}"/>
   </xacro:tiago_arm>
   <xacro:if value="${has_ft_sensor_right}">

Commit message: Add arm_left and arm_right params

File: tiago_dual_description/robots/tiago_dual.urdf.xacro (robot description, xacro)
@@ -9,4 +9,6 @@
 <robot  xmlns:xacro="http://ros.org/wiki/xacro"
         name="tiago_dual" >
+    <xacro:arg name="arm_left" default="true"/> <!-- true, false -->
+    <xacro:arg name="arm_right" default="true"/> <!-- true, false -->
     <xacro:arg name="end_effector_left" default="pal-hey5"/> <!-- pal-gripper, pal-hey5, schunk-wsg-->
     <xacro:arg name="end_effector_right" default="pal-hey5"/> <!-- pal-gripper, pal-hey5, schunk-wsg-->
@@ -17,4 +19,6 @@
     <xacro:arg name="multiple" default="false"/>
     <xacro:arg name="namespace" default=""/>
+    <xacro:property name="has_arm_left" value="$(arg arm_left)" />
+    <xacro:property name="has_arm_right" value="$(arg arm_right)" />
     <xacro:property name="end_effector_left" value="$(arg end_effector_left)" />
     <xacro:property name="end_effector_right" value="$(arg end_effector_right)" />
@@ -76,19 +80,23 @@
   <xacro:head name="head" parent="torso_lift_link" camera_model="$(arg camera_model)"/>
   <!-- Left -->
-  <xacro:tiago_arm name="arm_left" parent="torso_lift_link" wrist_6_range="${wrist_left_6_range}" reflect="-1" tiago_dual="1" arm_1_offset="${arm_left_1_joint_offset}" arm_2_offset="${arm_left_2_joint_offset}" arm_3_offset="${arm_left_3_joint_offset}" arm_4_offset="${arm_left_4_joint_offset}" arm_5_offset="${arm_left_5_joint_offset}" arm_6_offset="${arm_left_6_joint_offset}" arm_7_offset="${arm_left_7_joint_offset}">
-    <origin xyz="0.02556 0.19 -0.171" rpy="${180 * deg_to_rad} 0 ${90 * deg_to_rad}"/>
-  </xacro:tiago_arm>
-  <xacro:if value="${has_ft_sensor_left}">
-      <xacro:ft_sensor name="wrist_left" parent="arm_left_tool_link" />
+  <xacro:if value="${has_arm_left}">
+	  <xacro:tiago_arm name="arm_left" parent="torso_lift_link" wrist_6_range="${wrist_left_6_range}" reflect="-1" tiago_dual="1" arm_1_offset="${arm_left_1_joint_offset}" arm_2_offset="${arm_left_2_joint_offset}" arm_3_offset="${arm_left_3_joint_offset}" arm_4_offset="${arm_left_4_joint_offset}" arm_5_offset="${arm_left_5_joint_offset}" arm_6_offset="${arm_left_6_joint_offset}" arm_7_offset="${arm_left_7_joint_offset}">
+	    <origin xyz="0.02556 0.19 -0.171" rpy="${180 * deg_to_rad} 0 ${90 * deg_to_rad}"/>
+	  </xacro:tiago_arm>
+	  <xacro:if value="${has_ft_sensor_left}">
+	      <xacro:ft_sensor name="wrist_left" parent="arm_left_tool_link" />
+	  </xacro:if>
+  <xacro:tiago_end_effector name="${end_effector_left_name}" parent="${end_effector_left_link}" type="${end_effector_left}" reflect="-1"/>
   </xacro:if>
-  <xacro:tiago_end_effector name="${end_effector_left_name}" parent="${end_effector_left_link}" type="${end_effector_left}" reflect="-1"/>
   <!-- Right -->
-  <xacro:tiago_arm name="arm_right" parent="torso_lift_link" wrist_6_range="${wrist_right_6_range}" reflect="1" tiago_dual="1" arm_1_offset="${arm_right_1_joint_offset}" arm_2_offset="${arm_right_2_joint_offset}" arm_3_offset="${arm_right_3_joint_offset}" arm_4_offset="${arm_right_4_joint_offset}" arm_5_offset="${arm_right_5_joint_offset}" arm_6_offset="${arm_right_6_joint_offset}" arm_7_offset="${arm_right_7_joint_offset}">
-    <origin xyz="0.02556 -0.19 -0.171" rpy="0 0 ${-90 * deg_to_rad}"/>
-  </xacro:tiago_arm>
-  <xacro:if value="${has_ft_sensor_right}">
-      <xacro:ft_sensor name="wrist_right" parent="arm_right_tool_link" />
+  <xacro:if value="${has_arm_right}">
+	  <xacro:tiago_arm name="arm_right" parent="torso_lift_link" wrist_6_range="${wrist_right_6_range}" reflect="1" tiago_dual="1" arm_1_offset="${arm_right_1_joint_offset}" arm_2_offset="${arm_right_2_joint_offset}" arm_3_offset="${arm_right_3_joint_offset}" arm_4_offset="${arm_right_4_joint_offset}" arm_5_offset="${arm_right_5_joint_offset}" arm_6_offset="${arm_right_6_joint_offset}" arm_7_offset="${arm_right_7_joint_offset}">
+	    <origin xyz="0.02556 -0.19 -0.171" rpy="0 0 ${-90 * deg_to_rad}"/>
+	  </xacro:tiago_arm>
+	  <xacro:if value="${has_ft_sensor_right}">
+	      <xacro:ft_sensor name="wrist_right" parent="arm_right_tool_link" />
+	  </xacro:if>
+	  <xacro:tiago_end_effector name="${end_effector_right_name}" parent="${end_effector_right_link}" type="${end_effector_right}" reflect="1"/>
   </xacro:if>
-  <xacro:tiago_end_effector name="${end_effector_right_name}" parent="${end_effector_right_link}" type="${end_effector_right}" reflect="1"/>
   <!-- RGBD Laser Link -->
   <joint name="rgbd_laser_joint" type="fixed">

Commit message: Update arm_*_6 range based on the wrist type

File: tiago_dual_description/robots/tiago_dual.urdf.xacro (robot description, xacro)
@@ -11,4 +11,6 @@
     <xacro:arg name="arm_left" default="true"/> <!-- true, false -->
     <xacro:arg name="arm_right" default="true"/> <!-- true, false -->
+    <xacro:arg name="wrist_left_model" default="wrist-2010"/>
+    <xacro:arg name="wrist_right_model" default="wrist-2010"/>
     <xacro:arg name="end_effector_left" default="pal-hey5"/> <!-- pal-gripper, pal-hey5, schunk-wsg-->
     <xacro:arg name="end_effector_right" default="pal-hey5"/> <!-- pal-gripper, pal-hey5, schunk-wsg-->
@@ -54,6 +56,16 @@
    <xacro:property name="end_effector_right_link"       value="${'wrist_right_ft_tool_link' if has_ft_sensor_right else 'arm_right_tool_link'}"/>
    <xacro:property name="end_effector_right_name"       value="${'hand_right' if end_effector_right == 'pal-hey5' else 'gripper_right'}"/>
-   <xacro:property name="wrist_left_6_range"      value="${ 81 if has_ft_sensor_left else 90 }"/>
-   <xacro:property name="wrist_right_6_range"     value="${ 81 if has_ft_sensor_right else 90 }"/>
+   <xacro:if value="${wrist_left_model == 'wrist-2010'}">
+     <xacro:property name="wrist_left_6_range"           value="${ 81 if has_ft_sensor_left else 90 }"/>
+   </xacro:if>
+   <xacro:if value="${wrist_left_model == 'wrist-2017'}">
+     <xacro:property name="wrist_left_6_range"           value="81"/>
+   </xacro:if>
+   <xacro:if value="${wrist_right_model == 'wrist-2010'}">
+     <xacro:property name="wrist_right_6_range"           value="${ 81 if has_ft_sensor_right else 90 }"/>
+   </xacro:if>
+   <xacro:if value="${wrist_right_model == 'wrist-2017'}">
+     <xacro:property name="wrist_right_6_range"           value="81"/>
+   </xacro:if>
    <xacro:property name="head_link_name"          value="head_2_link"/>
   <!-- The following included files set up definitions of parts of the robot body -->

Commit message: added missing xacro properties

File: tiago_dual_description/robots/tiago_dual.urdf.xacro (robot description, xacro)
@@ -21,4 +21,6 @@
     <xacro:arg name="multiple" default="false"/>
     <xacro:arg name="namespace" default=""/>
+    <xacro:property name="wrist_left_model" value="$(arg wrist_left_model)" />
+    <xacro:property name="wrist_right_model" value="$(arg wrist_right_model)" />
     <xacro:property name="has_arm_left" value="$(arg arm_left)" />
     <xacro:property name="has_arm_right" value="$(arg arm_right)" />

Commit message: Change tool link position depending on wrist type

File: tiago_dual_description/robots/tiago_dual.urdf.xacro (robot description, xacro)
@@ -64,16 +64,4 @@
    <xacro:property name="end_effector_right_link"       value="${'wrist_right_ft_tool_link' if has_ft_sensor_right else 'arm_right_tool_link'}"/>
    <xacro:property name="end_effector_right_name"       value="${'hand_right' if end_effector_right == 'pal-hey5' else 'gripper_right'}"/>
-   <xacro:if value="${wrist_left_model == 'wrist-2010'}">
-     <xacro:property name="wrist_left_6_range"           value="${ 81 if has_ft_sensor_left else 90 }"/>
-   </xacro:if>
-   <xacro:if value="${wrist_left_model == 'wrist-2017'}">
-     <xacro:property name="wrist_left_6_range"           value="81"/>
-   </xacro:if>
-   <xacro:if value="${wrist_right_model == 'wrist-2010'}">
-     <xacro:property name="wrist_right_6_range"           value="${ 81 if has_ft_sensor_right else 90 }"/>
-   </xacro:if>
-   <xacro:if value="${wrist_right_model == 'wrist-2017'}">
-     <xacro:property name="wrist_right_6_range"           value="81"/>
-   </xacro:if>
    <xacro:property name="head_link_name"          value="head_2_link"/>
   <!-- The following included files set up definitions of parts of the robot body -->
@@ -101,5 +89,5 @@
   <!-- Left -->
   <xacro:if value="${has_arm_left}">
-	  <xacro:tiago_arm name="arm_left" parent="torso_lift_link" wrist_6_range="${wrist_left_6_range}" reflect="-1" tiago_dual="1" arm_1_offset="${arm_left_1_joint_offset}" arm_2_offset="${arm_left_2_joint_offset}" arm_3_offset="${arm_left_3_joint_offset}" arm_4_offset="${arm_left_4_joint_offset}" arm_5_offset="${arm_left_5_joint_offset}" arm_6_offset="${arm_left_6_joint_offset}" arm_7_offset="${arm_left_7_joint_offset}">
+	  <xacro:tiago_arm name="arm_left" parent="torso_lift_link" wrist_model="${wrist_left_model}" has_ft_sensor="${has_ft_sensor_left}" reflect="-1" tiago_dual="1" arm_1_offset="${arm_left_1_joint_offset}" arm_2_offset="${arm_left_2_joint_offset}" arm_3_offset="${arm_left_3_joint_offset}" arm_4_offset="${arm_left_4_joint_offset}" arm_5_offset="${arm_left_5_joint_offset}" arm_6_offset="${arm_left_6_joint_offset}" arm_7_offset="${arm_left_7_joint_offset}">
 	    <origin xyz="0.02556 0.19 -0.171" rpy="${180 * deg_to_rad} 0 ${90 * deg_to_rad}"/>
 	  </xacro:tiago_arm>
@@ -111,5 +99,5 @@
   <!-- Right -->
   <xacro:if value="${has_arm_right}">
-	  <xacro:tiago_arm name="arm_right" parent="torso_lift_link" wrist_6_range="${wrist_right_6_range}" reflect="1" tiago_dual="1" arm_1_offset="${arm_right_1_joint_offset}" arm_2_offset="${arm_right_2_joint_offset}" arm_3_offset="${arm_right_3_joint_offset}" arm_4_offset="${arm_right_4_joint_offset}" arm_5_offset="${arm_right_5_joint_offset}" arm_6_offset="${arm_right_6_joint_offset}" arm_7_offset="${arm_right_7_joint_offset}">
+	  <xacro:tiago_arm name="arm_right" parent="torso_lift_link" wrist_model="${wrist_right_model}" has_ft_sensor="${has_ft_sensor_right}" reflect="1" tiago_dual="1" arm_1_offset="${arm_right_1_joint_offset}" arm_2_offset="${arm_right_2_joint_offset}" arm_3_offset="${arm_right_3_joint_offset}" arm_4_offset="${arm_right_4_joint_offset}" arm_5_offset="${arm_right_5_joint_offset}" arm_6_offset="${arm_right_6_joint_offset}" arm_7_offset="${arm_right_7_joint_offset}">
 	    <origin xyz="0.02556 -0.19 -0.171" rpy="0 0 ${-90 * deg_to_rad}"/>
 	  </xacro:tiago_arm>

Commit message: pass the camera origin as an argument to head

File: tiago_dual_description/robots/tiago_dual.urdf.xacro (robot description, xacro)
@@ -86,5 +86,8 @@
   <xacro:base_sensors name="base" laser_model="$(arg laser_model)" sonars="true" microphone="true"/>
   <xacro:tiago_dual_torso name="torso" parent="base_link"/>
-  <xacro:head name="head" parent="torso_lift_link" camera_model="$(arg camera_model)"/>
+  <xacro:head name="head" parent="torso_lift_link" camera_model="$(arg camera_model)">
+    <!-- Camera origin Post Eye-Hand Calibration -->
+    <origin xyz="${camera_position_x} ${camera_position_y} ${camera_position_z}" rpy="${camera_orientation_r} ${camera_orientation_p} ${camera_orientation_y}" />
+  </xacro:head>
   <!-- Left -->
   <xacro:if value="${has_arm_left}">

Commit message: parse package name instead of individual elements and load files respective to package

File: tiago_dual_description/robots/tiago_dual.urdf.xacro (robot description, xacro)
@@ -86,8 +86,5 @@
   <xacro:base_sensors name="base" laser_model="$(arg laser_model)" sonars="true" microphone="true"/>
   <xacro:tiago_dual_torso name="torso" parent="base_link"/>
-  <xacro:head name="head" parent="torso_lift_link" camera_model="$(arg camera_model)">
-    <!-- Camera origin Post Eye-Hand Calibration -->
-    <origin xyz="${camera_position_x} ${camera_position_y} ${camera_position_z}" rpy="${camera_orientation_r} ${camera_orientation_p} ${camera_orientation_y}" />
-  </xacro:head>
+  <xacro:head name="head" parent="torso_lift_link" camera_model="$(arg camera_model)" description_calibration_package="tiago_dual_description_calibration"/>
   <!-- Left -->
   <xacro:if value="${has_arm_left}">
