Commit message: added changes to support tiago_dual with and without screen

File: tiago_dual_description/robots/tiago_dual.urdf.xacro (robot description, xacro)
@@ -19,4 +19,5 @@
     <xacro:arg name="laser_model" default="sick-571"/> <!-- false, hokuyo, sick-551, sick-561, sick-571-->
     <xacro:arg name="camera_model" default="orbbec-astra"/> <!-- false, orbbec-astra, orbbec-astra-pro, asus-xtion -->
+    <xacro:arg name="has_screen" default="false"/> <!-- true, false -->
     <xacro:arg name="multiple" default="false"/>
     <xacro:arg name="namespace" default=""/>
@@ -31,4 +32,5 @@
     <xacro:property name="laser_model" value="$(arg laser_model)" />
     <xacro:property name="camera_model" value="$(arg camera_model)" />
+    <xacro:property name="has_screen" value="$(arg has_screen)" />
     <xacro:property name="is_multiple" value="$(arg multiple)" />
     <xacro:property name="nsp" value="$(arg namespace)" />
@@ -85,5 +87,5 @@
   <!-- Now we can start using the macros included above to define the actual robot -->
   <xacro:base_sensors name="base" laser_model="$(arg laser_model)" sonars="true" microphone="true"/>
-  <xacro:tiago_dual_torso name="torso" parent="base_link"/>
+  <xacro:tiago_dual_torso name="torso" parent="base_link" has_screen="$(arg has_screen)"/>
   <xacro:head name="head" parent="torso_lift_link" camera_model="$(arg camera_model)" description_calibration_package="tiago_dual_description_calibration"/>
   <!-- Left -->

File: tiago_dual_description/urdf/torso/torso_dual.urdf.xacro (robot description, xacro)
@@ -14,5 +14,5 @@
   <xacro:property name="torso_max_vel"  value="0.07" />
   <xacro:property name="torso_eps"      value="0.02" />
-  <xacro:macro name="tiago_dual_torso" params="name parent">
+  <xacro:macro name="tiago_dual_torso" params="name parent has_screen">
   <!-- Bottom fixed part of column -->
   <link name="${name}_fixed_link">
@@ -92,41 +92,59 @@
     </inertial>
     <!-- Lifting body -->
-    <visual>
-      <origin rpy="0 0 0" xyz="0 0 0" />
-       <geometry>
-        <mesh filename="package://tiago_dual_description/meshes/torso/torso_lift_dual_arm.stl" scale="1 1 1"/>
-      </geometry>
-      <material name="White"/>
-    </visual>
-    <collision>
-      <origin rpy="0 0 0" xyz="0 0 0" />
-       <geometry>
-        <mesh filename="package://tiago_description/meshes/torso/torso_lift_collision_core.dae" scale="1 1 1"/>
-      </geometry>
-      <material name="LightGrey"/>
-    </collision>
-    <!-- left shoulder collision-->
-    <collision>
-      <origin rpy="0 0 0" xyz="-0.131 0.17 -0.02556" />
-       <geometry>
-        <mesh filename="package://tiago_description/meshes/torso/torso_lift_collision_shoulder.dae" scale="1 1 1"/>
-      </geometry>
-      <material name="LightGrey"/>
-    </collision>
-    <!-- right shoulder collision-->
-    <collision>
-      <origin rpy="0 0 0" xyz="-0.131 -0.19 -0.02556" />
-       <geometry>
-        <mesh filename="package://tiago_description/meshes/torso/torso_lift_collision_shoulder.dae" scale="1 1 1"/>
-      </geometry>
-      <material name="LightGrey"/>
-    </collision>
-    <collision>
-      <origin rpy="0 0 0" xyz="0 0 0" />
-       <geometry>
-        <mesh filename="package://tiago_description/meshes/torso/torso_lift_collision_neck.dae" scale="1 1 1"/>
-      </geometry>
-      <material name="LightGrey"/>
-    </collision>
+    <xacro:if value="${has_screen}">
+      <visual>
+        <origin rpy="0 0 0" xyz="0 0 0" />
+         <geometry>
+          <mesh filename="package://tiago_dual_description/meshes/torso/torso_lift_dual_arm_with_screen.stl" scale="1 1 1"/>
+        </geometry>
+        <material name="White"/>
+      </visual>
+      <collision>
+        <origin rpy="0 0 0" xyz="0 0 0" />
+         <geometry>
+          <mesh filename="package://tiago_dual_description/meshes/torso/torso_lift_dual_arm_with_screen.dae" scale="1 1 1"/>
+        </geometry>
+        <material name="LightGrey"/>
+      </collision>
+    </xacro:if>
+    <xacro:unless value="${has_screen}">
+      <visual>
+        <origin rpy="0 0 0" xyz="0 0 0" />
+         <geometry>
+          <mesh filename="package://tiago_dual_description/meshes/torso/torso_lift_dual_arm.stl" scale="1 1 1"/>
+        </geometry>
+        <material name="White"/>
+      </visual>
+      <collision>
+        <origin rpy="0 0 0" xyz="0 0 0" />
+         <geometry>
+          <mesh filename="package://tiago_description/meshes/torso/torso_lift_collision_core.dae" scale="1 1 1"/>
+        </geometry>
+        <material name="LightGrey"/>
+      </collision>
+      <!-- left shoulder collision-->
+      <collision>
+        <origin rpy="0 0 0" xyz="-0.131 0.17 -0.02556" />
+         <geometry>
+          <mesh filename="package://tiago_description/meshes/torso/torso_lift_collision_shoulder.dae" scale="1 1 1"/>
+        </geometry>
+        <material name="LightGrey"/>
+      </collision>
+      <!-- right shoulder collision-->
+      <collision>
+        <origin rpy="0 0 0" xyz="-0.131 -0.19 -0.02556" />
+         <geometry>
+          <mesh filename="package://tiago_description/meshes/torso/torso_lift_collision_shoulder.dae" scale="1 1 1"/>
+        </geometry>
+        <material name="LightGrey"/>
+      </collision>
+      <collision>
+        <origin rpy="0 0 0" xyz="0 0 0" />
+         <geometry>
+          <mesh filename="package://tiago_description/meshes/torso/torso_lift_collision_neck.dae" scale="1 1 1"/>
+        </geometry>
+        <material name="LightGrey"/>
+      </collision>
+    </xacro:unless>
   </link>
   <joint name="${name}_lift_joint" type="prismatic">

Commit message: Add master calibration to tiago dual

File: tiago_dual_description/robots/tiago_dual.urdf.xacro (robot description, xacro)
@@ -21,4 +21,5 @@
     <xacro:arg name="has_screen" default="false"/> <!-- true, false -->
     <xacro:arg name="multiple" default="false"/>
+    <xacro:arg name="description_calibration_file" default="$(find tiago_dual_description_calibration)/urdf/calibration/calibration_constants.urdf.xacro"/>
     <xacro:arg name="namespace" default=""/>
     <xacro:property name="wrist_left_model" value="$(arg wrist_left_model)" />
@@ -67,4 +68,5 @@
    <xacro:property name="end_effector_right_name"       value="${'hand_right' if end_effector_right == 'pal-hey5' else 'gripper_right'}"/>
    <xacro:property name="head_link_name"          value="head_2_link"/>
+   <xacro:property name="description_calibration_file"       value="${'$(find tiago_dual_description_calibration)/urdf/calibration/calibration_constants.urdf.xacro' if description_calibration_file == '' else description_calibration_file}"/>
   <!-- The following included files set up definitions of parts of the robot body -->
   <!-- Base -->
@@ -73,5 +75,5 @@
   <xacro:include filename="$(find tiago_dual_description)/urdf/torso/torso_dual.urdf.xacro" />
   <!-- Arm -->
-  <xacro:include filename="$(find tiago_dual_description_calibration)/urdf/calibration/calibration_constants.urdf.xacro" />
+  <xacro:include filename="$(arg description_calibration_file)" />
   <xacro:include filename="$(find tiago_description)/urdf/arm/arm.urdf.xacro" />
   <!-- End Effector -->

Commit message: Use optenv to get description calibration path

File: tiago_dual_description/robots/tiago_dual.urdf.xacro (robot description, xacro)
@@ -21,5 +21,5 @@
     <xacro:arg name="has_screen" default="false"/> <!-- true, false -->
     <xacro:arg name="multiple" default="false"/>
-    <xacro:arg name="description_calibration_file" default="$(find tiago_dual_description_calibration)/urdf/calibration/calibration_constants.urdf.xacro"/>
+    <xacro:arg name="description_calibration_dir" default="$(find tiago_dual_description_calibration)/urdf/calibration"/>
     <xacro:arg name="namespace" default=""/>
     <xacro:property name="wrist_left_model" value="$(arg wrist_left_model)" />
@@ -68,5 +68,5 @@
    <xacro:property name="end_effector_right_name"       value="${'hand_right' if end_effector_right == 'pal-hey5' else 'gripper_right'}"/>
    <xacro:property name="head_link_name"          value="head_2_link"/>
-   <xacro:property name="description_calibration_file"       value="${'$(find tiago_dual_description_calibration)/urdf/calibration/calibration_constants.urdf.xacro' if description_calibration_file == '' else description_calibration_file}"/>
+   <xacro:property name="description_calibration_dir"       value="${arg description_calibration_dir}"/>
   <!-- The following included files set up definitions of parts of the robot body -->
   <!-- Base -->
@@ -75,5 +75,5 @@
   <xacro:include filename="$(find tiago_dual_description)/urdf/torso/torso_dual.urdf.xacro" />
   <!-- Arm -->
-  <xacro:include filename="$(arg description_calibration_file)" />
+  <xacro:include filename="$(arg description_calibration_dir)/calibration_constants.urdf.xacro" />
   <xacro:include filename="$(find tiago_description)/urdf/arm/arm.urdf.xacro" />
   <!-- End Effector -->

Commit message: Add no_safety_eps param

File: tiago_dual_description/robots/tiago_dual.urdf.xacro (robot description, xacro)
@@ -37,4 +37,5 @@
     <xacro:property name="is_multiple" value="$(arg multiple)" />
     <xacro:property name="nsp" value="$(arg namespace)" />
+    <xacro:property name="no_safety_eps" value="$(arg no_safety_eps)" />
   <xacro:if value="${wrist_left_model not in ['wrist-2010', 'wrist-2017']}">
     <xacro:wrong_wrist_model/>
@@ -96,5 +97,5 @@
   <!-- Left -->
   <xacro:if value="${has_arm_left}">
-	  <xacro:tiago_arm name="arm_left" parent="torso_lift_link" wrist_model="${wrist_left_model}" has_ft_sensor="${has_ft_sensor_left}" reflect="-1" tiago_dual="1" arm_1_offset="${arm_left_1_joint_offset}" arm_2_offset="${arm_left_2_joint_offset}" arm_3_offset="${arm_left_3_joint_offset}" arm_4_offset="${arm_left_4_joint_offset}" arm_5_offset="${arm_left_5_joint_offset}" arm_6_offset="${arm_left_6_joint_offset}" arm_7_offset="${arm_left_7_joint_offset}">
+	  <xacro:tiago_arm name="arm_left" parent="torso_lift_link" wrist_model="${wrist_left_model}" has_ft_sensor="${has_ft_sensor_left}" reflect="-1" tiago_dual="1" arm_1_offset="${arm_left_1_joint_offset}" arm_2_offset="${arm_left_2_joint_offset}" arm_3_offset="${arm_left_3_joint_offset}" arm_4_offset="${arm_left_4_joint_offset}" arm_5_offset="${arm_left_5_joint_offset}" arm_6_offset="${arm_left_6_joint_offset}" arm_7_offset="${arm_left_7_joint_offset}" no_safety_eps="${no_safety_eps}">
 	    <origin xyz="0.02556 0.19 -0.171" rpy="${180 * deg_to_rad} 0 ${90 * deg_to_rad}"/>
 	  </xacro:tiago_arm>
@@ -106,5 +107,5 @@
   <!-- Right -->
   <xacro:if value="${has_arm_right}">
-	  <xacro:tiago_arm name="arm_right" parent="torso_lift_link" wrist_model="${wrist_right_model}" has_ft_sensor="${has_ft_sensor_right}" reflect="1" tiago_dual="1" arm_1_offset="${arm_right_1_joint_offset}" arm_2_offset="${arm_right_2_joint_offset}" arm_3_offset="${arm_right_3_joint_offset}" arm_4_offset="${arm_right_4_joint_offset}" arm_5_offset="${arm_right_5_joint_offset}" arm_6_offset="${arm_right_6_joint_offset}" arm_7_offset="${arm_right_7_joint_offset}">
+	  <xacro:tiago_arm name="arm_right" parent="torso_lift_link" wrist_model="${wrist_right_model}" has_ft_sensor="${has_ft_sensor_right}" reflect="1" tiago_dual="1" arm_1_offset="${arm_right_1_joint_offset}" arm_2_offset="${arm_right_2_joint_offset}" arm_3_offset="${arm_right_3_joint_offset}" arm_4_offset="${arm_right_4_joint_offset}" arm_5_offset="${arm_right_5_joint_offset}" arm_6_offset="${arm_right_6_joint_offset}" arm_7_offset="${arm_right_7_joint_offset}"  no_safety_eps="${no_safety_eps}">
 	    <origin xyz="0.02556 -0.19 -0.171" rpy="0 0 ${-90 * deg_to_rad}"/>
 	  </xacro:tiago_arm>

Commit message: Creating tiago dual with omni base robot

File: tiago_dual_description/robots/tiago_dual.urdf.xacro (robot description, xacro)
@@ -21,4 +21,5 @@
     <xacro:arg name="has_screen" default="false"/> <!-- true, false -->
     <xacro:arg name="multiple" default="false"/>
+    <xacro:arg name="base_type" default="pmb2"/> <!-- pmb2, omni_base -->
     <xacro:arg name="description_calibration_dir" default="$(find tiago_dual_description_calibration)/urdf/calibration"/>
     <xacro:arg name="extrinsic_calibration_dir" default="$(find tiago_dual_description_calibration)/urdf/calibration"/>
@@ -35,4 +36,5 @@
     <xacro:property name="camera_model" value="$(arg camera_model)" />
     <xacro:property name="has_screen" value="$(arg has_screen)" />
+    <xacro:property name="base_type" value="$(arg base_type)" />
     <xacro:property name="is_multiple" value="$(arg multiple)" />
     <xacro:property name="nsp" value="$(arg namespace)" />
@@ -62,4 +64,7 @@
     <xacro:wrong_camera_model/>
   </xacro:if>
+  <xacro:if value="${base_type not in ['pmb2', 'omni_base']}">
+    <xacro:wrong_base_type/>
+  </xacro:if>
    <xacro:property name="has_schunk_ft"           value="${ft_sensor == 'schunk-ft'}"/>
    <xacro:property name="has_ft_sensor_left"      value="${ft_sensor_left == 'schunk-ft'}"/> <!-- This should be OR'ed with other FT sensors-->
@@ -73,5 +78,5 @@
   <!-- The following included files set up definitions of parts of the robot body -->
   <!-- Base -->
-  <xacro:include filename="$(find pmb2_description)/urdf/base/base_sensors.urdf.xacro" />
+  <xacro:include filename="$(find ${base_type}_description)/urdf/base/base_sensors.urdf.xacro" />
   <!-- Torso -->
   <xacro:include filename="$(find tiago_dual_description)/urdf/torso/torso_dual.urdf.xacro" />
@@ -90,5 +95,10 @@
   <xacro:include filename="$(find tiago_description)/urdf/materials.urdf.xacro" />
   <!-- Now we can start using the macros included above to define the actual robot -->
-  <xacro:base_sensors name="base" laser_model="$(arg laser_model)" sonars="true" microphone="true"/>
+  <xacro:if value="${base_type == 'pmb2'}">
+    <xacro:base_sensors name="base" laser_model="$(arg laser_model)" sonars="true" microphone="true"/>
+  </xacro:if>
+  <xacro:if value="${base_type == 'omni_base'}">
+    <xacro:base_sensors name="base" front_laser_model="$(arg laser_model)" rear_laser_model="$(arg laser_model)"/>
+  </xacro:if>
   <xacro:tiago_dual_torso name="torso" parent="base_link" has_screen="$(arg has_screen)"/>
   <xacro:head name="head" parent="torso_lift_link" camera_model="$(arg camera_model)"

Commit message: generate new config files

File: tiago_dual_description/robots/tiago_dual.urdf.xacro (robot description, xacro)
@@ -70,6 +70,8 @@
    <xacro:property name="has_ft_sensor_left"      value="${ft_sensor_left == 'schunk-ft'}"/> <!-- This should be OR'ed with other FT sensors-->
    <xacro:property name="has_ft_sensor_right"     value="${ft_sensor_right == 'schunk-ft'}"/> <!-- This should be OR'ed with other FT sensors-->
+   <xacro:property name="has_end_effector_left"        value="${end_effector_left != 'false'}"/>
    <xacro:property name="end_effector_left_link"       value="${'wrist_left_ft_tool_link' if has_ft_sensor_left else 'arm_left_tool_link'}"/>
    <xacro:property name="end_effector_left_name"       value="${'hand_left' if end_effector_left == 'pal-hey5' else 'gripper_left'}"/>
+   <xacro:property name="has_end_effector_right"        value="${end_effector_right != 'false'}"/>
    <xacro:property name="end_effector_right_link"       value="${'wrist_right_ft_tool_link' if has_ft_sensor_right else 'arm_right_tool_link'}"/>
    <xacro:property name="end_effector_right_name"       value="${'hand_right' if end_effector_right == 'pal-hey5' else 'gripper_right'}"/>
@@ -114,5 +116,6 @@
 	      <xacro:ft_sensor name="wrist_left" parent="arm_left_tool_link" />
 	  </xacro:if>
-  <xacro:tiago_end_effector name="${end_effector_left_name}" parent="${end_effector_left_link}" type="${end_effector_left}" reflect="-1" is_dual="true"/>
+  <xacro:tiago_end_effector name="${end_effector_left_name}" parent="${end_effector_left_link}" type="${end_effector_left}"
+    has_end_effector="${has_end_effector_left}" reflect="-1" is_dual="true"/>
   </xacro:if>
   <!-- Right -->
@@ -124,5 +127,5 @@
 	      <xacro:ft_sensor name="wrist_right" parent="arm_right_tool_link" />
 	  </xacro:if>
-	  <xacro:tiago_end_effector name="${end_effector_right_name}" parent="${end_effector_right_link}" type="${end_effector_right}" reflect="1" is_dual="true"/>
+	  <xacro:tiago_end_effector name="${end_effector_right_name}" parent="${end_effector_right_link}" type="${end_effector_right}" has_end_effector="${has_end_effector_right}" reflect="1" is_dual="true"/>
   </xacro:if>
   <!-- RGBD Laser Link -->

Commit message: correctly update tiago_dual.urdf.xacro

File: tiago_dual_description/robots/tiago_dual.urdf.xacro (robot description, xacro)
@@ -71,6 +71,8 @@
    <xacro:property name="has_ft_sensor_left"      value="${ft_sensor_left == 'schunk-ft'}"/> <!-- This should be OR'ed with other FT sensors-->
    <xacro:property name="has_ft_sensor_right"     value="${ft_sensor_right == 'schunk-ft'}"/> <!-- This should be OR'ed with other FT sensors-->
+   <xacro:property name="has_end_effector_left"        value="${end_effector_left != 'false'}"/>
    <xacro:property name="end_effector_left_link"       value="${'wrist_left_ft_tool_link' if has_ft_sensor_left else 'arm_left_tool_link'}"/>
    <xacro:property name="end_effector_left_name"       value="${'hand_left' if end_effector_left == 'pal-hey5' else 'gripper_left'}"/>
+   <xacro:property name="has_end_effector_right"        value="${end_effector_right != 'false'}"/>
    <xacro:property name="end_effector_right_link"       value="${'wrist_right_ft_tool_link' if has_ft_sensor_right else 'arm_right_tool_link'}"/>
    <xacro:property name="end_effector_right_name"       value="${'hand_right' if end_effector_right == 'pal-hey5' else 'gripper_right'}"/>
@@ -115,5 +117,6 @@
 	      <xacro:ft_sensor name="wrist_left" parent="arm_left_tool_link" />
 	  </xacro:if>
-  <xacro:tiago_end_effector name="${end_effector_left_name}" parent="${end_effector_left_link}" type="${end_effector_left}" reflect="-1" is_dual="true"/>
+  <xacro:tiago_end_effector name="${end_effector_left_name}" parent="${end_effector_left_link}" type="${end_effector_left}"
+    has_end_effector="${has_end_effector_left}" reflect="-1" is_dual="true"/>
   </xacro:if>
   <!-- Right -->
@@ -125,5 +128,5 @@
 	      <xacro:ft_sensor name="wrist_right" parent="arm_right_tool_link" />
 	  </xacro:if>
-	  <xacro:tiago_end_effector name="${end_effector_right_name}" parent="${end_effector_right_link}" type="${end_effector_right}" reflect="1" is_dual="true"/>
+	  <xacro:tiago_end_effector name="${end_effector_right_name}" parent="${end_effector_right_link}" type="${end_effector_right}" has_end_effector="${has_end_effector_right}" reflect="1" is_dual="true"/>
   </xacro:if>
   <!-- RGBD Laser Link -->

Commit message: file_suffix consistency

File: tiago_dual_description/robots/tiago_dual.urdf.xacro (robot description, xacro)
@@ -71,8 +71,8 @@
    <xacro:property name="has_ft_sensor_left"      value="${ft_sensor_left == 'schunk-ft'}"/> <!-- This should be OR'ed with other FT sensors-->
    <xacro:property name="has_ft_sensor_right"     value="${ft_sensor_right == 'schunk-ft'}"/> <!-- This should be OR'ed with other FT sensors-->
-   <xacro:property name="has_end_effector_left"        value="${end_effector_left != 'false'}"/>
+   <xacro:property name="has_end_effector_left"        value="${end_effector_left not in ['false', 'False', 'no-ee']}"/>
    <xacro:property name="end_effector_left_link"       value="${'wrist_left_ft_tool_link' if has_ft_sensor_left else 'arm_left_tool_link'}"/>
    <xacro:property name="end_effector_left_name"       value="${'hand_left' if end_effector_left == 'pal-hey5' else 'gripper_left'}"/>
-   <xacro:property name="has_end_effector_right"        value="${end_effector_right != 'false'}"/>
+   <xacro:property name="has_end_effector_right"        value="${end_effector_right not in ['false', 'False', 'no-ee']}"/>
    <xacro:property name="end_effector_right_link"       value="${'wrist_right_ft_tool_link' if has_ft_sensor_right else 'arm_right_tool_link'}"/>
    <xacro:property name="end_effector_right_name"       value="${'hand_right' if end_effector_right == 'pal-hey5' else 'gripper_right'}"/>

Commit message: Added parameter to main xacro

File: tiago_dual_description/robots/tiago_dual.urdf.xacro (robot description, xacro)
@@ -25,4 +25,5 @@
     <xacro:arg name="extrinsic_calibration_dir" default="$(find tiago_dual_description_calibration)/urdf/calibration"/>
     <xacro:arg name="namespace" default=""/>
+    <xacro:arg name="fixed_torso" default="false" />
     <xacro:arg name="no_safety_eps" default="false"/>
     <xacro:property name="wrist_left_model" value="$(arg wrist_left_model)" />
@@ -41,4 +42,5 @@
     <xacro:property name="nsp" value="$(arg namespace)" />
     <xacro:property name="no_safety_eps" value="$(arg no_safety_eps)" />
+    <xacro:property name="fixed_torso" value="$(arg fixed_torso)" />
   <xacro:if value="${wrist_left_model not in ['wrist-2010', 'wrist-2017']}">
     <xacro:wrong_wrist_model/>

Commit message: Uncomment parts of the urdf

File: tiago_dual_description/robots/tiago_dual.urdf.xacro (robot description, xacro)
@@ -116,5 +116,4 @@
   <xacro:tiago_dual_ros2_control
     use_sim="$(arg use_sim)" />
-<xacro:property name="M_PI" value="3.1415926535897931" />
   <!-- Now we can start using the macros included above to define the actual robot -->
   <xacro:if value="${base_type == 'pmb2'}">

File: tiago_dual_description/urdf/torso/torso_dual.urdf.xacro (robot description, xacro)
@@ -91,4 +91,7 @@
       <origin xyz="0.04361 -0.00116 -0.17334" rpy="0.00000 0.00000 0.00000"/>
       <mass value="9.594213"/>
+      <!-- <inertia ixx="0.24487000000" ixy="-0.00145600000" ixz="-0.00974200000"
+               iyy="0.24926900000" iyz="0.00828100000"
+               izz="0.09039500000"/> -->
       <inertia ixx="0.326395" ixy="-0.000844" ixz="-0.018905"
                iyy="0.235332" iyz="0.009042"

Commit message: make possible to choose the control period for gazebo

File: tiago_dual_description/robots/tiago_dual.urdf.xacro (robot description, xacro)
@@ -27,4 +27,5 @@
     <xacro:arg name="fixed_torso" default="false" />
     <xacro:arg name="no_safety_eps" default="false"/>
+    <xacro:arg name="gazebo_control_period" default="0.001"/> <!-- 1000Hz or 100 Hz-->
     <xacro:property name="wrist_left_model" value="$(arg wrist_left_model)" />
     <xacro:property name="wrist_right_model" value="$(arg wrist_right_model)" />
@@ -43,4 +44,5 @@
     <xacro:property name="no_safety_eps" value="$(arg no_safety_eps)" />
     <xacro:property name="fixed_torso" value="$(arg fixed_torso)" />
+    <xacro:property name="gazebo_control_period" value="$(arg gazebo_control_period)" />
   <xacro:if value="${wrist_left_model not in ['wrist-2010', 'wrist-2017']}">
     <xacro:wrong_wrist_model/>
