Commit message: Fix the height between base_link and torso for the omni_base

File: tiago_dual_description/robots/tiago_dual.urdf.xacro (robot description, xacro)
@@ -163,5 +163,12 @@
   </xacro:if>
   <!-- Torso -->
-  <xacro:tiago_dual_torso name="torso" parent="base_link" has_screen="${has_screen}"/>
+  <xacro:tiago_dual_torso name="torso" parent="base_link" has_screen="${has_screen}">
+    <xacro:if value="${base_type == 'pmb2'}">
+      <origin rpy="0 0 0" xyz="-0.062 0.0 0.193" />
+    </xacro:if>
+    <xacro:if value="${base_type == 'omni_base'}">
+      <origin rpy="0 0 0" xyz="-0.062 0.0 0.215" />
+    </xacro:if>
+  </xacro:tiago_dual_torso>
   <!-- Left arm -->
   <xacro:if value="${has_arm_left}">

File: tiago_dual_description/urdf/torso/torso_dual.urdf.xacro (robot description, xacro)
@@ -19,5 +19,5 @@
   <xacro:include filename="$(find pal_urdf_utils)/urdf/deg_to_rad.urdf.xacro" />
   <!-- MACRO DEFINITION -->
-  <xacro:macro name="tiago_dual_torso" params="name parent has_screen">
+  <xacro:macro name="tiago_dual_torso" params="name parent *origin has_screen">
     <!-- Bottom fixed part of column -->
     <link name="${name}_fixed_link">
@@ -48,5 +48,5 @@
     </link>
     <joint name="${name}_fixed_joint" type="fixed">
-      <origin rpy="0 0 0" xyz="-0.062 0.0 0.193" />
+      <xacro:insert_block name="origin"/>
       <parent link="${parent}" />
       <child link="${name}_fixed_link" />
@@ -79,5 +79,5 @@
     </gazebo>
     <joint name="${name}_fixed_column_joint" type="fixed">
-      <origin rpy="0 0 0" xyz="-0.062 0 0.195" />
+      <xacro:insert_block name="origin"/>
       <parent link="${parent}" />
       <child link="${name}_fixed_column_link" />

Commit message: Load master calibration data

File: tiago_dual_description/robots/tiago_dual.urdf.xacro (robot description, xacro)
@@ -52,6 +52,6 @@
   <xacro:arg name="no_safety_eps" default="false"/>
   <!-- Calibration -->
-  <xacro:arg name="description_calibration_dir" default="$(find tiago_dual_description)/urdf/calibration"/>
-  <xacro:arg name="extrinsic_calibration_dir" default="$(find tiago_dual_description)/urdf/calibration"/>
+  <xacro:arg name="eye_hand_calibration_dir" default="$(find tiago_dual_description)/urdf/calibration"/>
+  <xacro:arg name="camera_extrinsic_calibration_dir" default="$(find tiago_dual_description)/urdf/calibration"/>
   <!-- Execution env config -->
   <xacro:arg name="use_sim_time" default="false"/>
@@ -121,6 +121,6 @@
   <xacro:property name="end_effector_right_name" value="${'hand_right' if end_effector_right == 'pal-hey5' else 'gripper_right'}"/>
   <!-- Calibration -->
-  <xacro:property name="description_calibration_dir" value="$(arg description_calibration_dir)"/>
-  <xacro:property name="extrinsic_calibration_dir" value="$(arg extrinsic_calibration_dir)"/>
+  <xacro:property name="eye_hand_calibration_dir" value="$(arg eye_hand_calibration_dir)"/>
+  <xacro:property name="camera_extrinsic_calibration_dir" value="$(arg camera_extrinsic_calibration_dir)"/>
   <!-- Execution env configuration -->
   <xacro:property name="use_sim_time" default="$(arg use_sim_time)"/>

File: tiago_dual_description/ros2_control/ros2_control.urdf.xacro (robot description, xacro)
@@ -18,5 +18,5 @@
   <xacro:include filename="$(find ${base_type}_description)/urdf/wheels/wheel.ros2_control.xacro" />
   <xacro:include filename="$(find ${base_type}_description)/urdf/sensors/sensors.ros2_control.xacro" />
-  <xacro:include filename="${description_calibration_dir}/calibration_constants.urdf.xacro" />
+  <xacro:include filename="${eye_hand_calibration_dir}/eye_hand_calibration.urdf.xacro" />
   <!-- Arm, FT, EE -->
   <xacro:if value="${has_arm_right or has_arm_left}">

File: tiago_dual_description/urdf/calibration/camera_extrinsic_calibration.urdf.xacro (robot description, xacro)
@@ -1,17 +1,17 @@
 <?xml version="1.0"?>
 <!--
-  Copyright (c) 2024 PAL Robotics S.L. All rights reserved.
-  Licensed under the Apache License, Version 2.0 (the "License");
-  you may not use this file except in compliance with the License.
-  You may obtain a copy of the License at
-      http://www.apache.org/licenses/LICENSE-2.0
-  Unless required by applicable law or agreed to in writing, software
-  distributed under the License is distributed on an "AS IS" BASIS,
-  WITHOUT WARRANTIES OR CONDITIONS OF ANY KIND, either express or implied.
-  See the License for the specific language governing permissions and
-  limitations under the License.
+Copyright (c) 2024 PAL Robotics S.L. All rights reserved.
+Licensed under the Apache License, Version 2.0 (the "License");
+you may not use this file except in compliance with the License.
+You may obtain a copy of the License at
+    http://www.apache.org/licenses/LICENSE-2.0
+Unless required by applicable law or agreed to in writing, software
+distributed under the License is distributed on an "AS IS" BASIS,
+WITHOUT WARRANTIES OR CONDITIONS OF ANY KIND, either express or implied.
+See the License for the specific language governing permissions and
+limitations under the License.
  -->
 <robot xmlns:xacro="http://ros.org/wiki/xacro">
-  <!--INCLUDES-->
+  <!-- INCLUDES -->
   <xacro:include filename="$(find pal_urdf_utils)/urdf/deg_to_rad.urdf.xacro" />
   <!-- MACRO DEFINITION -->

File: tiago_dual_description/urdf/calibration/eye_hand_calibration.urdf.xacro (robot description, xacro)
@@ -13,4 +13,6 @@
  -->
 <robot xmlns:xacro="http://ros.org/wiki/xacro">
+  <!-- INCLUDES -->
+  <xacro:include filename="$(find pal_urdf_utils)/urdf/deg_to_rad.urdf.xacro" />
   <!-- PROPERTIES -->
   <xacro:property name="camera_position_x" value="0.0908" />
@@ -36,5 +38,3 @@
   <xacro:property name="head_1_joint_offset" value="0.0" />
   <xacro:property name="head_2_joint_offset" value="0.0" />
-  <!-- INCLUDES -->
-  <xacro:include filename="$(find pal_urdf_utils)/urdf/deg_to_rad.urdf.xacro" />
 </robot>

Commit message: Add velodyne params + mesh

File: tiago_dual_description/robots/tiago_dual.urdf.xacro (robot description, xacro)
@@ -27,4 +27,5 @@
     <xacro:arg name="fixed_torso" default="false" />
     <xacro:arg name="no_safety_eps" default="false"/>
+    <xacro:arg name="has_velodyne" default="false" />
     <xacro:arg name="gazebo_control_period" default="0.001"/> <!-- 1000Hz or 100 Hz-->
     <xacro:property name="wrist_left_model" value="$(arg wrist_left_model)" />
@@ -43,4 +44,5 @@
     <xacro:property name="nsp" value="$(arg namespace)" />
     <xacro:property name="no_safety_eps" value="$(arg no_safety_eps)" />
+    <xacro:property name="has_velodyne" value="$(arg has_velodyne)" />
     <xacro:property name="fixed_torso" value="$(arg fixed_torso)" />
     <xacro:property name="gazebo_control_period" value="$(arg gazebo_control_period)" />
@@ -110,5 +112,5 @@
     <xacro:base_sensors name="base" front_laser_model="$(arg laser_model)" rear_laser_model="$(arg laser_model)"/>
   </xacro:if>
-  <xacro:tiago_dual_torso name="torso" parent="base_link" has_screen="$(arg has_screen)"/>
+  <xacro:tiago_dual_torso name="torso" parent="base_link" base_type="$(arg base_type)" has_screen="$(arg has_screen)" has_velodyne="$(arg has_velodyne)" />
   <xacro:head name="head" parent="torso_lift_link" camera_model="$(arg camera_model)"
 	  description_calibration_dir="$(arg description_calibration_dir)"

File: tiago_dual_description/urdf/torso/torso_dual.urdf.xacro (robot description, xacro)
@@ -13,5 +13,5 @@
   <xacro:property name="torso_max_vel"  value="0.07" />
   <xacro:property name="torso_eps"      value="0.02" />
-  <xacro:macro name="tiago_dual_torso" params="name parent has_screen">
+  <xacro:macro name="tiago_dual_torso" params="name parent base_type has_screen has_velodyne">
   <!-- Bottom fixed part of column -->
   <link name="${name}_fixed_link">
@@ -23,24 +23,76 @@
                izz="0.07699800000"/>
     </inertial>
-    <visual>
-      <origin rpy="0 0 0" xyz="0 0 0" />
-      <geometry>
-        <mesh filename="package://tiago_dual_description/meshes/torso/torso_fix.stl" scale="1 1 1"/>
-      </geometry>
-      <material name="LightGrey"/>
-    </visual>
-    <collision>
-      <origin rpy="0 0 0" xyz="0.09 0.0 0.02" />
-      <geometry>
-        <box size="0.4 0.28 0.075"/>
-      </geometry>
-    </collision>
-    <collision>
-      <origin rpy="0 0 0" xyz="0 0 0.05" />
-      <geometry>
-        <box size="0.25 0.265 0.052"/>
-      </geometry>
-    </collision>
+    <xacro:if value="${has_velodyne}">
+      <xacro:if value="${base_type == 'pmb2'}">
+        <!-- TODO: Integrate the torso_fix_with_velodyne_pmb2.stl -->
+      </xacro:if>
+      <xacro:if value="${base_type == 'omni_base'}">
+        <visual>
+          <origin rpy="0 0 0" xyz="0 0 0" />
+          <geometry>
+            <mesh filename="package://tiago_dual_description/meshes/torso/torso_fix_with_velodyne.stl" scale="1 1 1"/>
+          </geometry>
+          <material name="White"/>
+        </visual>
+        <collision>
+          <origin rpy="0 0 0" xyz="0.129898 0.0 0.035888" />
+          <geometry>
+            <box size="0.482507 0.262781 0.07314"/>
+          </geometry>
+        </collision>
+        <collision>
+          <origin rpy="0 0 0" xyz="0.005267 0 0.041713" />
+          <geometry>
+            <box size="0.232581 0.262781 0.084366"/>
+          </geometry>
+        </collision>
+        <collision>
+          <origin rpy="0 0 0" xyz="0.277349 0.0 0.083478" />
+          <geometry>
+            <cylinder radius="0.07" length="0.10"/>
+          </geometry>
+        </collision>
+      </xacro:if>
+    </xacro:if>
+    <xacro:unless value="${has_velodyne}">
+      <visual>
+        <origin rpy="0 0 0" xyz="0 0 0" />
+        <geometry>
+          <mesh filename="package://tiago_dual_description/meshes/torso/torso_fix.stl" scale="1 1 1"/>
+        </geometry>
+        <material name="LightGrey"/>
+      </visual>
+      <collision>
+        <origin rpy="0 0 0" xyz="0.085 0.0 0.035" />
+        <geometry>
+          <box size="0.43 0.295 0.056"/>
+        </geometry>
+      </collision>
+      <collision>
+        <origin rpy="0 0 0" xyz="0 0 0.065" />
+        <geometry>
+          <box size="0.263 0.295 0.117"/>
+        </geometry>
+      </collision>
+    </xacro:unless>
   </link>
+  <xacro:if value="${has_velodyne}">
+    <xacro:if value="${base_type == 'pmb2'}">
+      <!-- TODO: Change it accordingly to the new model for pmb2 -->
+    </xacro:if>
+    <xacro:if value="${base_type == 'omni_base'}">
+      <link name="${name}_velodyne_link"/>
+      <joint name="${name}_velodyne_joint" type="fixed">
+        <origin rpy="0 0 0" xyz="0.277 0.0 0.0523" />
+        <parent link="${name}_fixed_link" />
+        <child link="${name}_velodyne_link" />
+        <axis xyz="0 0 0" />
+      </joint>
+      <xacro:include filename="$(find velodyne_description)/urdf/VLP-16.urdf.xacro"/>
+      <xacro:VLP-16 parent="${name}_velodyne_link" name="velodyne" topic="velodyne_points" organize_cloud="true" hz="1" samples="440" gpu="false">
+        <origin xyz="0 0 0" rpy="0 0 0" />
+      </xacro:VLP-16>
+    </xacro:if>
+  </xacro:if>
   <joint name="${name}_fixed_joint" type="fixed">
     <origin rpy="0 0 0" xyz="-0.062 0.0 0.193" />

Commit message: Add gazebo_version xacro argument

File: tiago_dual_description/robots/tiago_dual.urdf.xacro (robot description, xacro)
@@ -59,4 +59,5 @@
   <xacro:arg name="namespace" default=""/>
   <xacro:arg name="is_public_sim" default="false"/>
+  <xacro:arg name="gazebo_version" default="classic"/>
   <!-- PROPERTIES -->
   <!-- HW configuration -->
@@ -128,4 +129,5 @@
   <xacro:property name="namespace" value="$(arg namespace)" />
   <xacro:property name="is_public_sim" value="$(arg is_public_sim)" />
+  <xacro:property name="gazebo_version" value="$(arg gazebo_version)" />
   <!-- INCLUDES -->
   <!-- Tools -->

Commit message: add calibration_tool parameter

File: tiago_dual_description/robots/tiago_dual.urdf.xacro (robot description, xacro)
@@ -51,4 +51,6 @@
   <!-- false, true -->
   <xacro:arg name="no_safety_eps" default="false"/>
+  <!-- False, True -->
+  <xacro:arg name="calibration_tool" default="False" />
   <!-- Calibration -->
   <xacro:arg name="eye_hand_calibration_dir" default="$(find tiago_dual_description)/urdf/calibration"/>
@@ -76,4 +78,5 @@
   <xacro:property name="has_screen" value="$(arg has_screen)" />
   <xacro:property name="no_safety_eps" value="$(arg no_safety_eps)" />
+  <xacro:property name="calibration_tool" value="$(arg calibration_tool)"/>
   <!-- HW configuration check -->
   <xacro:if value="${base_type not in ['pmb2', 'omni_base']}">
