Commit message: Add support for new gazebo

File: tiago_dual_description/ros2_control/ros2_control.urdf.xacro (robot description, xacro)
@@ -44,7 +44,16 @@
     <xacro:if value="${use_sim_time}">
       <gazebo>
-        <plugin filename="libgazebo_ros2_control.so" name="gazebo_ros2_control">
-          <parameters>$(find tiago_description)/ros2_control/gazebo_controller_manager_cfg.yaml</parameters>
-        </plugin>
+        <xacro:if value="${gazebo_version == 'classic'}">
+          <plugin filename="libgazebo_ros2_control.so" name="gazebo_ros2_control">
+            <parameters>$(find tiago_dual_description)/ros2_control/gazebo_controller_manager_cfg.yaml</parameters>
+          </plugin>
+        </xacro:if>
+        <xacro:if value="${gazebo_version == 'gazebo'}">
+          <plugin filename="gz_ros2_control-system" name="gz_ros2_control::GazeboSimROS2ControlPlugin">
+            <robot_param>robot_description</robot_param>
+            <robot_param_node>robot_state_publisher</robot_param_node>
+            <parameters>$(find tiago_dual_description)/ros2_control/gazebo_controller_manager_cfg.yaml</parameters>
+          </plugin>
+        </xacro:if>
       </gazebo>
     </xacro:if>
@@ -54,5 +63,10 @@
       <hardware>
         <xacro:if value="${use_sim_time}">
-          <plugin>gazebo_ros2_control/GazeboSystem</plugin>
+          <xacro:if value="${gazebo_version == 'classic'}">
+            <plugin>gazebo_ros2_control/GazeboSystem</plugin>
+          </xacro:if>
+          <xacro:if value="${gazebo_version == 'gazebo'}">
+            <plugin>gz_ros2_control/GazeboSimSystem</plugin>
+          </xacro:if>
         </xacro:if>
         <xacro:unless value="${use_sim_time}">

File: tiago_dual_description/urdf/torso/torso_dual.urdf.xacro (robot description, xacro)
@@ -148,4 +148,12 @@
       </xacro:unless>
     </link>
+    <!-- TODO: set lower limit back to 0 when moving to Gazebo Harmonic or ROS 2 Jazzy -->
+    <!-- See https://github.com/gazebosim/gz-sim/issues/1684 for more information -->
+    <xacro:if value="${gazebo_version == 'classic'}">
+      <xacro:property name="torso_lower_limit" value="0.0"/>
+    </xacro:if>
+    <xacro:if value="${gazebo_version == 'gazebo'}">
+      <xacro:property name="torso_lower_limit" value="-1e-3"/>
+    </xacro:if>
     <joint name="${name}_lift_joint" type="prismatic">
       <origin rpy="0.0 0.0 0.0" xyz="0.0 0.0 0.597" />
@@ -153,5 +161,5 @@
       <child link="${name}_lift_link" />
       <axis xyz="0 0 1" />
-      <limit effort="2000" lower="0" upper="0.35" velocity="${torso_max_vel}" />
+      <limit effort="2000" lower="${torso_lower_limit}" upper="0.35" velocity="${torso_max_vel}" />
       <calibration rising="0.0" />
       <dynamics damping="1000" />
